Commit message: 添加gitignore以忽略模型文件

File: catkin_ws/src/multi_robot_scenario/xacro/go2/robot.xacro (robot description, xacro)
@@ -31,4 +31,5 @@
     <!-- Actually, the rotor will rotate and the joint is not fixed. Reduction ratio should be considered. -->
     <!-- Debug mode will hung up the robot, use "true" or "false" to switch it. -->
+    <!-- 删除部分 -->
     <xacro:if value="$(arg DEBUG)">
         <link name="world"/>
@@ -40,10 +41,10 @@
     </xacro:if>
     <link name="base">
-        <visual>
+        <!-- <visual>
             <origin rpy="0 0 0" xyz="0 0 0"/>
             <geometry>
                 <box size="0.001 0.001 0.001"/>
             </geometry>
-        </visual>
+        </visual> -->
     </link>
     <joint name="floating_base" type="fixed">
